File: extras/schematic/basic_sachematic.brd (EAGLE design)
At the start: 41.1 x 49.8 mm, 15 parts, among them X1 1501_03

Commit message: Extras
Parts:
- C7: value (none) -> 100nF
Changed lines of the file:
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@@
 <attribute name="VALUE" x="-82.77" y="-16.851" size="1.27" layer="27" ratio="10"/>
 </element>
-<element name="C7" library="rcl" library_urn="urn:adsk.eagle:library:334" package="C1825K" package3d_urn="urn:adsk.eagle:package:23684/2" value="" x="-87.625" y="-14.5" smashed="yes">
+<element name="C7" library="rcl" library_urn="urn:adsk.eagle:library:334" package="C1825K" package3d_urn="urn:adsk.eagle:package:23684/2" value="100nF" x="-87.625" y="-14.5" smashed="yes">
 <attribute name="NAME" x="-89.225" y="-10.95" size="1.016" layer="25"/>
 <attribute name="SPICEPREFIX" value="C" x="-87.625" y="-14.5" size="1.778" layer="27" display="off"/>

Commit message: KT0915 Arduino Library
Parts:
- renumbered KT1 to KT0915
Changed lines of the file:
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@@
 <drawing>
 <settings>
-<setting alwaysvectorfont="no"/>
+<setting alwaysvectorfont="yes"/>
 <setting keepoldvectorfont="yes"/>
 <setting verticaltext="up"/>
@@
 </autorouter>
 <elements>
-<element name="KT1" library="dp_devices" package="KT0915" value="" x="9.6875" y="30.0625" smashed="yes" rot="R90">
+<element name="KT0915" library="dp_devices" package="KT0915" value="" x="9.6875" y="30.0625" smashed="yes" rot="R90">
 <attribute name="NAME" x="11.6875" y="27.0625" size="1.27" layer="25" font="vector" ratio="10" rot="R180"/>
 <attribute name="VALUE" x="11.6875" y="34.1875" size="1.27" layer="27" font="vector" ratio="10" rot="R180"/>
@@
 <signals>
 <signal name="N$12">
-<contactref element="KT1" pad="RFINP"/>
+<contactref element="KT0915" pad="RFINP"/>
 <wire x1="3" y1="30.5" x2="6.75" y2="30.5" width="0.254" layer="1"/>
 <wire x1="6.75" y1="30.5" x2="6.9085" y2="30.3795" width="0.254" layer="1"/>
@@
 </signal>
 <signal name="N$26">
-<contactref element="KT1" pad="ROUT"/>
+<contactref element="KT0915" pad="ROUT"/>
 <wire x1="10.25" y1="29.25" x2="12.25" y2="29.25" width="0.254" layer="1"/>
 <wire x1="10.25" y1="37.25" x2="10.25" y2="29.25" width="0.254" layer="1"/>
@@
 </signal>
 <signal name="GND">
-<contactref element="KT1" pad="AVSS"/>
+<contactref element="KT0915" pad="AVSS"/>
 <contactref element="ARDUINO1" pad="GND@1"/>
 <contactref element="ARDUINO1" pad="GND@2"/>
@@
 <contactref element="X1" pad="1"/>
 <contactref element="C7" pad="1"/>
-<contactref element="KT1" pad="RFGND"/>
+<contactref element="KT0915" pad="RFGND"/>
 <contactref element="C3" pad="2"/>
 <contactref element="C4" pad="2"/>
-<contactref element="KT1" pad="DVSS"/>
+<contactref element="KT0915" pad="DVSS"/>
 <wire x1="-86.125" y1="-24.6875" x2="-86.125" y2="-34.875" width="0" layer="19" extent="1-1"/>
 <wire x1="-89.125" y1="-14.5" x2="-86.125" y2="-24.6875" width="0" layer="19" extent="1-1"/>
@@
 <signal name="N$2">
 <contactref element="ARDUINO1" pad="A4"/>
-<contactref element="KT1" pad="SDA"/>
+<contactref element="KT0915" pad="SDA"/>
 <contactref element="R1" pad="2"/>
 <wire x1="-13.985" y1="16.21" x2="-78.9825" y2="-43.375" width="0" layer="19" extent="1-1"/>
@@
 <signal name="N$3">
 <contactref element="ARDUINO1" pad="A5"/>
-<contactref element="KT1" pad="SCL"/>
+<contactref element="KT0915" pad="SCL"/>
 <contactref element="R2" pad="2"/>
 <wire x1="-13.985" y1="18.75" x2="-78.9825" y2="-48" width="0" layer="19" extent="1-1"/>
@@
 <contactref element="C1" pad="1"/>
 <contactref element="C2" pad="1"/>
-<contactref element="KT1" pad="AVDD"/>
-<contactref element="KT1" pad="ENABLE"/>
+<contactref element="KT0915" pad="AVDD"/>
+<contactref element="KT0915" pad="ENABLE"/>
 <contactref element="R1" pad="1"/>
 <contactref element="R2" pad="1"/>
@@
 </signal>
 <signal name="N$4">
-<contactref element="KT1" pad="XI/RCLK"/>
+<contactref element="KT0915" pad="XI/RCLK"/>
 <contactref element="Q1" pad="2"/>
 <contactref element="C4" pad="1"/>
@@
 </signal>
 <signal name="N$5">
-<contactref element="KT1" pad="XO"/>
+<contactref element="KT0915" pad="XO"/>
 <contactref element="Q1" pad="1"/>
 <contactref element="C3" pad="1"/>
@@
 </signal>
 <signal name="N$6">
-<contactref element="KT1" pad="LOUT"/>
+<contactref element="KT0915" pad="LOUT"/>
 <contactref element="C6" pad="1"/>
 <wire x1="12.4665" y1="29.7445" x2="-72.4375" y2="-2.125" width="0" layer="19" extent="1-1"/>
@@
 </signal>
 <signal name="N$9">
-<contactref element="KT1" pad="AMINN"/>
+<contactref element="KT0915" pad="AMINN"/>
 <contactref element="C7" pad="2"/>
 <wire x1="6.9085" y1="31.6495" x2="-86.125" y2="-14.5" width="0" layer="19" extent="1-1"/>
 </signal>
 <signal name="N$11">
-<contactref element="KT1" pad="AMINP"/>
+<contactref element="KT0915" pad="AMINP"/>
 <contactref element="ANT1" pad="1"/>
 <wire x1="6.9085" y1="31.0145" x2="-81.5" y2="-12.1875" width="0" layer="19" extent="1-1"/>
