File: extras/schematic/minimal_receiver.brd (EAGLE design)
At the start: 41.1 x 49.8 mm, 15 parts, among them X1 1501_03

Commit message: KT0915 Arduino Library
Parts:
- added AM, DOWN, FM, UP: (no value), adafruit:TACT_PANA-EVQ
- C7: value (none) -> 100nF
- renumbered KT1 to KT0915
Connections:
- new net N$1: ARDUINO1.D4, FM.P$2
- new net N$10: AM.P$2, ARDUINO1.D5
- new net N$13: ARDUINO1.D6, UP.P$2
- new net N$14: ARDUINO1.D7, DOWN.P$2
- net GND: now also AM.P$1, DOWN.P$1, FM.P$1, KT0915.DVSS, UP.P$1
Changed lines of the file:
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@@
 <drawing>
 <settings>
-<setting alwaysvectorfont="no"/>
+<setting alwaysvectorfont="yes"/>
 <setting keepoldvectorfont="yes"/>
 <setting verticaltext="up"/>
@@
 </autorouter>
 <elements>
-<element name="KT1" library="dp_devices" package="KT0915" value="" x="9.6875" y="30.0625" smashed="yes" rot="R90">
+<element name="KT0915" library="dp_devices" package="KT0915" value="" x="9.6875" y="30.0625" smashed="yes" rot="R90">
 <attribute name="NAME" x="11.6875" y="27.0625" size="1.27" layer="25" font="vector" ratio="10" rot="R180"/>
 <attribute name="VALUE" x="11.6875" y="34.1875" size="1.27" layer="27" font="vector" ratio="10" rot="R180"/>
@@
 <attribute name="VALUE" x="-82.77" y="-16.851" size="1.27" layer="27" ratio="10"/>
 </element>
-<element name="C7" library="rcl" library_urn="urn:adsk.eagle:library:334" package="C1825K" package3d_urn="urn:adsk.eagle:package:23684/2" value="" x="-87.625" y="-14.5" smashed="yes">
+<element name="C7" library="rcl" library_urn="urn:adsk.eagle:library:334" package="C1825K" package3d_urn="urn:adsk.eagle:package:23684/2" value="100nF" x="-87.625" y="-14.5" smashed="yes">
 <attribute name="NAME" x="-89.225" y="-10.95" size="1.016" layer="25"/>
 <attribute name="SPICEPREFIX" value="C" x="-87.625" y="-14.5" size="1.778" layer="27" display="off"/>
@@
 <attribute name="VALUE" x="-87.1931" y="-50.775" size="1.27" layer="27" ratio="10"/>
 </element>
+<element name="FM" library="adafruit" library_urn="urn:adsk.eagle:library:420" package="TACT_PANA-EVQ" package3d_urn="urn:adsk.eagle:package:6240957/1" value="" x="-85.5" y="-54.625" smashed="yes">
+<attribute name="NAME" x="-88.543" y="-52.455" size="0.8128" layer="25" ratio="18"/>
+<attribute name="VALUE" x="-88.516" y="-57.076" size="0.4064" layer="27" ratio="10"/>
+</element>
+<element name="AM" library="adafruit" library_urn="urn:adsk.eagle:library:420" package="TACT_PANA-EVQ" package3d_urn="urn:adsk.eagle:package:6240957/1" value="" x="-85.5" y="-59.9375" smashed="yes">
+<attribute name="NAME" x="-88.543" y="-57.7675" size="0.8128" layer="25" ratio="18"/>
+<attribute name="VALUE" x="-88.516" y="-62.3885" size="0.4064" layer="27" ratio="10"/>
+</element>
+<element name="UP" library="adafruit" library_urn="urn:adsk.eagle:library:420" package="TACT_PANA-EVQ" package3d_urn="urn:adsk.eagle:package:6240957/1" value="" x="-85.5" y="-65.25" smashed="yes">
+<attribute name="NAME" x="-88.543" y="-63.08" size="0.8128" layer="25" ratio="18"/>
+<attribute name="VALUE" x="-88.516" y="-67.701" size="0.4064" layer="27" ratio="10"/>
+</element>
+<element name="DOWN" library="adafruit" library_urn="urn:adsk.eagle:library:420" package="TACT_PANA-EVQ" package3d_urn="urn:adsk.eagle:package:6240957/1" value="" x="-85.5" y="-70.5625" smashed="yes">
+<attribute name="NAME" x="-88.543" y="-68.3925" size="0.8128" layer="25" ratio="18"/>
+<attribute name="VALUE" x="-88.516" y="-73.0135" size="0.4064" layer="27" ratio="10"/>
+</element>
 </elements>
 <signals>
 <signal name="N$12">
-<contactref element="KT1" pad="RFINP"/>
+<contactref element="KT0915" pad="RFINP"/>
 <wire x1="3" y1="30.5" x2="6.75" y2="30.5" width="0.254" layer="1"/>
 <wire x1="6.75" y1="30.5" x2="6.9085" y2="30.3795" width="0.254" layer="1"/>
@@
 </signal>
 <signal name="N$26">
-<contactref element="KT1" pad="ROUT"/>
+<contactref element="KT0915" pad="ROUT"/>
 <wire x1="10.25" y1="29.25" x2="12.25" y2="29.25" width="0.254" layer="1"/>
 <wire x1="10.25" y1="37.25" x2="10.25" y2="29.25" width="0.254" layer="1"/>
@@
 </signal>
 <signal name="GND">
-<contactref element="KT1" pad="AVSS"/>
+<contactref element="KT0915" pad="AVSS"/>
 <contactref element="ARDUINO1" pad="GND@1"/>
 <contactref element="ARDUINO1" pad="GND@2"/>
@@
 <contactref element="X1" pad="1"/>
 <contactref element="C7" pad="1"/>
-<contactref element="KT1" pad="RFGND"/>
+<contactref element="KT0915" pad="RFGND"/>
 <contactref element="C3" pad="2"/>
 <contactref element="C4" pad="2"/>
+<contactref element="KT0915" pad="DVSS"/>
+<contactref element="FM" pad="P$1"/>
+<contactref element="AM" pad="P$1"/>
+<contactref element="UP" pad="P$1"/>
+<contactref element="DOWN" pad="P$1"/>
+<wire x1="-88.75" y1="-65.25" x2="-88.75" y2="-70.5625" width="0" layer="19" extent="1-1"/>
+<wire x1="-88.75" y1="-59.9375" x2="-88.75" y2="-65.25" width="0" layer="19" extent="1-1"/>
+<wire x1="-88.75" y1="-54.625" x2="-88.75" y2="-59.9375" width="0" layer="19" extent="1-1"/>
+<wire x1="-86.125" y1="-34.875" x2="-88.75" y2="-54.625" width="0" layer="19" extent="1-1"/>
 <wire x1="-86.125" y1="-24.6875" x2="-86.125" y2="-34.875" width="0" layer="19" extent="1-1"/>
 <wire x1="-89.125" y1="-14.5" x2="-86.125" y2="-24.6875" width="0" layer="19" extent="1-1"/>
@@
 <wire x1="6.9085" y1="29.7445" x2="-11.445" y2="25.1" width="0" layer="19" extent="1-1"/>
 <wire x1="12.4665" y1="30.3795" x2="6.9085" y2="29.7445" width="0" layer="19" extent="1-1"/>
+<wire x1="12.4665" y1="28.4745" x2="12.4665" y2="30.3795" width="0" layer="19" extent="1-1"/>
 </signal>
 <signal name="N$2">
 <contactref element="ARDUINO1" pad="A4"/>
-<contactref element="KT1" pad="SDA"/>
+<contactref element="KT0915" pad="SDA"/>
 <contactref element="R1" pad="2"/>
 <wire x1="-13.985" y1="16.21" x2="-78.9825" y2="-43.375" width="0" layer="19" extent="1-1"/>
@@
 <signal name="N$3">
 <contactref element="ARDUINO1" pad="A5"/>
-<contactref element="KT1" pad="SCL"/>
+<contactref element="KT0915" pad="SCL"/>
 <contactref element="R2" pad="2"/>
 <wire x1="-13.985" y1="18.75" x2="-78.9825" y2="-48" width="0" layer="19" extent="1-1"/>
@@
 <contactref element="C1" pad="1"/>
 <contactref element="C2" pad="1"/>
-<contactref element="KT1" pad="AVDD"/>
-<contactref element="KT1" pad="ENABLE"/>
+<contactref element="KT0915" pad="AVDD"/>
+<contactref element="KT0915" pad="ENABLE"/>
 <contactref element="R1" pad="1"/>
 <contactref element="R2" pad="1"/>
@@
 </signal>
 <signal name="N$4">
-<contactref element="KT1" pad="XI/RCLK"/>
+<contactref element="KT0915" pad="XI/RCLK"/>
 <contactref element="Q1" pad="2"/>
 <contactref element="C4" pad="1"/>
@@
 </signal>
 <signal name="N$5">
-<contactref element="KT1" pad="XO"/>
+<contactref element="KT0915" pad="XO"/>
 <contactref element="Q1" pad="1"/>
 <contactref element="C3" pad="1"/>
@@
 </signal>
 <signal name="N$6">
-<contactref element="KT1" pad="LOUT"/>
+<contactref element="KT0915" pad="LOUT"/>
 <contactref element="C6" pad="1"/>
 <wire x1="12.4665" y1="29.7445" x2="-72.4375" y2="-2.125" width="0" layer="19" extent="1-1"/>
@@
 </signal>
 <signal name="N$9">
-<contactref element="KT1" pad="AMINN"/>
+<contactref element="KT0915" pad="AMINN"/>
 <contactref element="C7" pad="2"/>
 <wire x1="6.9085" y1="31.6495" x2="-86.125" y2="-14.5" width="0" layer="19" extent="1-1"/>
 </signal>
 <signal name="N$11">
-<contactref element="KT1" pad="AMINP"/>
+<contactref element="KT0915" pad="AMINP"/>
 <contactref element="ANT1" pad="1"/>
 <wire x1="6.9085" y1="31.0145" x2="-81.5" y2="-12.1875" width="0" layer="19" extent="1-1"/>
 </signal>
+<signal name="N$1">
+<contactref element="ARDUINO1" pad="D4"/>
+<contactref element="FM" pad="P$2"/>
+<wire x1="-26.685" y1="12.4" x2="-82.25" y2="-54.625" width="0" layer="19" extent="1-1"/>
+</signal>
+<signal name="N$10">
+<contactref element="ARDUINO1" pad="D5"/>
+<contactref element="AM" pad="P$2"/>
+<wire x1="-26.685" y1="9.86" x2="-82.25" y2="-59.9375" width="0" layer="19" extent="1-1"/>
+</signal>
+<signal name="N$13">
+<contactref element="ARDUINO1" pad="D6"/>
+<contactref element="UP" pad="P$2"/>
+<wire x1="-26.685" y1="7.32" x2="-82.25" y2="-65.25" width="0" layer="19" extent="1-1"/>
+</signal>
+<signal name="N$14">
+<contactref element="ARDUINO1" pad="D7"/>
+<contactref element="DOWN" pad="P$2"/>
+<wire x1="-26.685" y1="4.78" x2="-82.25" y2="-70.5625" width="0" layer="19" extent="1-1"/>
+</signal>
 </signals>
