File: extras/schematic/OLED_FM_AM_SW_receiver.brd (EAGLE design)
At the start: 41.1 x 49.8 mm, 15 parts, among them X1 1501_03

Commit message: KT0915 Arduino Library
Parts:
- added SW1: Band Up, adafruit:TACT_PANA-EVQ
- added SW2: Band Down, adafruit:TACT_PANA-EVQ
- added SW3: Tune Up, adafruit:TACT_PANA-EVQ
- added SW4: Tune Down, adafruit:TACT_PANA-EVQ
- added SW5: Am Bandwidth, adafruit:TACT_PANA-EVQ
- added SW6: Audio Gain, adafruit:TACT_PANA-EVQ
- added U$1: DISPLAY-OLED-128X64-I2C, diy-modules:DISPLAY-OLED-128X64-I2C
- ARDUINO1: value (none) -> ProMini 3.3v 8MHz
- C7: value (none) -> 100nF
- renumbered KT1 to KT0915
Connections:
- new net N$1: ARDUINO1.D4, SW1.P$2
- new net N$10: ARDUINO1.D5, SW2.P$2
- new net N$13: ARDUINO1.D6, SW3.P$2
- new net N$14: ARDUINO1.D7, SW4.P$2
- net GND: now also KT0915.DVSS, SW1.P$1, SW2.P$1, SW3.P$1, SW4.P$1, SW5.P$1, SW6.P$1, U$1.1
- net N$2: now also U$1.4
- net N$3: now also U$1.3
- net VCC: now also U$1.2

Commit message: KT0915 Arduino Library
Parts:
- SW3: value Tune Up -> Vol Up
- SW4: value Tune Down -> Vol Down
- renumbered U$1 to OLED1
Connections:
- new net N$15: ARDUINO1.D8, SW5.P$2
- new net N$16: ARDUINO1.D9, SW6.P$2
- new net N$17: OLED1.1, SW1.P$1, SW2.P$1, SW3.P$1, SW4.P$1, SW5.P$1, SW6.P$1
- net GND: no longer OLED1.1, SW1.P$1, SW2.P$1, SW3.P$1, SW4.P$1, SW5.P$1, SW6.P$1
Changed lines of the file:
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@@
 <attribute name="VALUE" x="-88.516" y="-62.3885" size="0.4064" layer="27" ratio="10"/>
 </element>
-<element name="SW3" library="adafruit" library_urn="urn:adsk.eagle:library:420" package="TACT_PANA-EVQ" package3d_urn="urn:adsk.eagle:package:6240957/1" value="Tune Up" x="-85.5" y="-65.25" smashed="yes">
+<element name="SW3" library="adafruit" library_urn="urn:adsk.eagle:library:420" package="TACT_PANA-EVQ" package3d_urn="urn:adsk.eagle:package:6240957/1" value="Vol Up" x="-85.5" y="-65.25" smashed="yes">
 <attribute name="NAME" x="-88.543" y="-63.08" size="0.8128" layer="25" ratio="18"/>
 <attribute name="VALUE" x="-88.516" y="-67.701" size="0.4064" layer="27" ratio="10"/>
 </element>
-<element name="SW4" library="adafruit" library_urn="urn:adsk.eagle:library:420" package="TACT_PANA-EVQ" package3d_urn="urn:adsk.eagle:package:6240957/1" value="Tune Down" x="-85.5" y="-70.5625" smashed="yes">
+<element name="SW4" library="adafruit" library_urn="urn:adsk.eagle:library:420" package="TACT_PANA-EVQ" package3d_urn="urn:adsk.eagle:package:6240957/1" value="Vol Down" x="-85.5" y="-70.5625" smashed="yes">
 <attribute name="NAME" x="-88.543" y="-68.3925" size="0.8128" layer="25" ratio="18"/>
 <attribute name="VALUE" x="-88.516" y="-73.0135" size="0.4064" layer="27" ratio="10"/>
@@
 <attribute name="VALUE" x="-88.516" y="-83.6385" size="0.4064" layer="27" ratio="10"/>
 </element>
-<element name="U$1" library="diy-modules" package="DISPLAY-OLED-128X64-I2C" value="DISPLAY-OLED-128X64-I2C" x="-103.8125" y="-67.1875" smashed="yes">
+<element name="OLED1" library="diy-modules" package="DISPLAY-OLED-128X64-I2C" value="DISPLAY-OLED-128X64-I2C" x="-103.8125" y="-67.1875" smashed="yes">
 <attribute name="NAME" x="-103.8125" y="-51.9475" size="1.27" layer="25" align="bottom-center"/>
 <attribute name="VALUE" x="-103.8125" y="-82.4275" size="1.27" layer="27" align="top-center"/>
@@
 <contactref element="C4" pad="2"/>
 <contactref element="KT0915" pad="DVSS"/>
-<contactref element="SW6" pad="P$1"/>
-<contactref element="SW1" pad="P$1"/>
-<contactref element="SW2" pad="P$1"/>
-<contactref element="SW3" pad="P$1"/>
-<contactref element="SW4" pad="P$1"/>
-<contactref element="SW5" pad="P$1"/>
-<contactref element="U$1" pad="1"/>
-<wire x1="-88.75" y1="-75.875" x2="-88.75" y2="-81.1875" width="0" layer="19" extent="1-1"/>
-<wire x1="-88.75" y1="-70.5625" x2="-88.75" y2="-75.875" width="0" layer="19" extent="1-1"/>
-<wire x1="-88.75" y1="-65.25" x2="-88.75" y2="-70.5625" width="0" layer="19" extent="1-1"/>
-<wire x1="-88.75" y1="-59.9375" x2="-88.75" y2="-65.25" width="0" layer="19" extent="1-1"/>
-<wire x1="-88.75" y1="-54.625" x2="-88.75" y2="-59.9375" width="0" layer="19" extent="1-1"/>
-<wire x1="-107.6225" y1="-54.4875" x2="-88.75" y2="-54.625" width="0" layer="19" extent="1-1"/>
-<wire x1="-86.125" y1="-34.875" x2="-88.75" y2="-54.625" width="0" layer="19" extent="1-1"/>
 <wire x1="-86.125" y1="-24.6875" x2="-86.125" y2="-34.875" width="0" layer="19" extent="1-1"/>
 <wire x1="-89.125" y1="-14.5" x2="-86.125" y2="-24.6875" width="0" layer="19" extent="1-1"/>
@@
 <contactref element="KT0915" pad="SDA"/>
 <contactref element="R1" pad="2"/>
-<contactref element="U$1" pad="4"/>
+<contactref element="OLED1" pad="4"/>
 <wire x1="-78.9825" y1="-43.375" x2="-100.0025" y2="-54.4875" width="0" layer="19" extent="1-1"/>
 <wire x1="-13.985" y1="16.21" x2="-78.9825" y2="-43.375" width="0" layer="19" extent="1-1"/>
@@
 </signal>
 <signal name="N$3">
-<contactref element="ARDUINO1" pad="A5"/>
 <contactref element="KT0915" pad="SCL"/>
 <contactref element="R2" pad="2"/>
-<contactref element="U$1" pad="3"/>
+<contactref element="OLED1" pad="3"/>
+<contactref element="ARDUINO1" pad="A5"/>
 <wire x1="-78.9825" y1="-48" x2="-102.5425" y2="-54.4875" width="0" layer="19" extent="1-1"/>
 <wire x1="-13.985" y1="18.75" x2="-78.9825" y2="-48" width="0" layer="19" extent="1-1"/>
@@
 <contactref element="R1" pad="1"/>
 <contactref element="R2" pad="1"/>
-<contactref element="U$1" pad="2"/>
+<contactref element="OLED1" pad="2"/>
 <wire x1="-89.1425" y1="-48" x2="-105.0825" y2="-54.4875" width="0" layer="19" extent="1-1"/>
 <wire x1="-89.1425" y1="-43.375" x2="-89.1425" y2="-48" width="0" layer="19" extent="1-1"/>
@@
 <wire x1="-26.685" y1="9.86" x2="-82.25" y2="-59.9375" width="0" layer="19" extent="1-1"/>
 </signal>
-<signal name="N$13">
+<signal name="N$14">
 <contactref element="ARDUINO1" pad="D6"/>
 <contactref element="SW3" pad="P$2"/>
 <wire x1="-26.685" y1="7.32" x2="-82.25" y2="-65.25" width="0" layer="19" extent="1-1"/>
 </signal>
-<signal name="N$14">
+<signal name="N$13">
 <contactref element="ARDUINO1" pad="D7"/>
 <contactref element="SW4" pad="P$2"/>
 <wire x1="-26.685" y1="4.78" x2="-82.25" y2="-70.5625" width="0" layer="19" extent="1-1"/>
 </signal>
+<signal name="N$15">
+<contactref element="ARDUINO1" pad="D8"/>
+<contactref element="SW5" pad="P$2"/>
+<wire x1="-26.685" y1="2.24" x2="-82.25" y2="-75.875" width="0" layer="19" extent="1-1"/>
+</signal>
+<signal name="N$16">
+<contactref element="ARDUINO1" pad="D9"/>
+<contactref element="SW6" pad="P$2"/>
+<wire x1="-26.685" y1="-0.3" x2="-82.25" y2="-81.1875" width="0" layer="19" extent="1-1"/>
+</signal>
+<signal name="N$17">
+<contactref element="OLED1" pad="1"/>
+<contactref element="SW6" pad="P$1"/>
+<contactref element="SW1" pad="P$1"/>
+<contactref element="SW2" pad="P$1"/>
+<contactref element="SW3" pad="P$1"/>
+<contactref element="SW4" pad="P$1"/>
+<contactref element="SW5" pad="P$1"/>
+<wire x1="-88.75" y1="-75.875" x2="-88.75" y2="-81.1875" width="0" layer="19" extent="1-1"/>
+<wire x1="-88.75" y1="-70.5625" x2="-88.75" y2="-75.875" width="0" layer="19" extent="1-1"/>
+<wire x1="-88.75" y1="-65.25" x2="-88.75" y2="-70.5625" width="0" layer="19" extent="1-1"/>
+<wire x1="-88.75" y1="-59.9375" x2="-88.75" y2="-65.25" width="0" layer="19" extent="1-1"/>
+<wire x1="-88.75" y1="-54.625" x2="-88.75" y2="-59.9375" width="0" layer="19" extent="1-1"/>
+<wire x1="-107.6225" y1="-54.4875" x2="-88.75" y2="-54.625" width="0" layer="19" extent="1-1"/>
+</signal>
 </signals>
