File: extras/schematic/OLED_FM_AM_SW_receiver.sch (EAGLE design)
At the start: 15 parts, among them X1 1501_03

Commit message: KT0915 Arduino Library
Parts:
- removed KT1: (no value), dp_devices:KT0915
- added KT0915: (no value), dp_devices:KT0915
- added SW1: Band Up, adafruit:SWITCH_PUSHBUTTONEVQ-PE
- added SW2: Band Down, adafruit:SWITCH_PUSHBUTTONEVQ-PE
- added SW3: Tune Up, adafruit:SWITCH_PUSHBUTTONEVQ-PE
- added SW4: Tune Down, adafruit:SWITCH_PUSHBUTTONEVQ-PE
- added SW5: Am Bandwidth, adafruit:SWITCH_PUSHBUTTONEVQ-PE
- added SW6: Audio Gain, adafruit:SWITCH_PUSHBUTTONEVQ-PE
- added U$1: DISPLAY-OLED-128X64-I2C, diy-modules:DISPLAY-OLED-128X64-I2C
- ARDUINO1: value (none) -> ProMini 3.3v 8MHz
- C7: value (none) -> 100nF
Connections:
- new net N$1: ARDUINO1.D4, SW1.P$2
- new net N$10: ARDUINO1.D5, SW2.P$2
- new net N$13: ARDUINO1.D6, SW3.P$2
- new net N$14: ARDUINO1.D7, SW4.P$2
- net GND: now also KT0915.AVSS, KT0915.DVSS, KT0915.RFGND, SW1.P$1, SW2.P$1, SW3.P$1, SW4.P$1, SW5.P$1, SW6.P$1, U$1.GND; no longer KT1.AVSS, KT1.DVSS, KT1.RFGND
- net N$11: now also KT0915.AMINP; no longer KT1.AMINP
- net N$12: now also KT0915.RFINP; no longer KT1.RFINP
- net N$2: now also KT0915.SDA, U$1.SDA; no longer KT1.SDA
- net N$26: now also KT0915.ROUT; no longer KT1.ROUT
- net N$3: now also KT0915.SCL, U$1.SCL; no longer KT1.SCL
- net N$4: now also KT0915.XI/RCLK; no longer KT1.XI/RCLK
- net N$5: now also KT0915.XO; no longer KT1.XO
- net N$6: now also KT0915.LOUT; no longer KT1.LOUT
- net N$9: now also KT0915.AMINN; no longer KT1.AMINN
- net VCC: now also KT0915.AVDD, KT0915.ENABLE, U$1.VCC; no longer KT1.AVDD, KT1.ENABLE
Other:
- moved on the sheet: ANT1, ANT2, C1, C2, C3, C4, C5, C6, C7, Q1, R1, R2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

Commit message: KT0915 Arduino Library
Parts:
- SW3: value Tune Up -> Vol Up
- SW4: value Tune Down -> Vol Down
- renumbered U$1 to OLED1
Connections:
- new net N$15: ARDUINO1.D8, SW5.P$2
- new net N$16: ARDUINO1.D9, SW6.P$2
- new net N$17: OLED1.GND, SW1.P$1, SW2.P$1, SW3.P$1, SW4.P$1, SW5.P$1, SW6.P$1
- net GND: no longer OLED1.GND, SW1.P$1, SW2.P$1, SW3.P$1, SW4.P$1, SW5.P$1, SW6.P$1
Other:
- moved on the sheet: SW1, SW2, SW3, SW4, SW5, SW6
