File: extras/schematic/basic_sachematic.sch (EAGLE design)
At the start: 15 parts, among them X1 1501_03

Commit message: Extras
Parts:
- C7: value (none) -> 100nF
Changed lines of the file:
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@@
 <part name="ANT1" library="discrete" library_urn="urn:adsk.eagle:library:211" deviceset="ANTENNA" device="" package3d_urn="urn:adsk.eagle:package:12928/1" value="AM Antenna"/>
 <part name="ANT2" library="discrete" library_urn="urn:adsk.eagle:library:211" deviceset="ANTENNA" device="" package3d_urn="urn:adsk.eagle:package:12928/1" value="FM Antenna"/>
-<part name="C7" library="rcl" library_urn="urn:adsk.eagle:library:334" deviceset="C-EU" device="C1825K" package3d_urn="urn:adsk.eagle:package:23684/2"/>
+<part name="C7" library="rcl" library_urn="urn:adsk.eagle:library:334" deviceset="C-EU" device="C1825K" package3d_urn="urn:adsk.eagle:package:23684/2" value="100nF"/>
 <part name="GND5" library="supply1" library_urn="urn:adsk.eagle:library:371" deviceset="GND" device=""/>
 <part name="SUPPLY3" library="supply2" library_urn="urn:adsk.eagle:library:372" deviceset="VCC" device=""/>

Commit message: KT0915 Arduino Library
Parts:
- renumbered KT1 to KT0915
Changed lines of the file:
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@@
 <drawing>
 <settings>
-<setting alwaysvectorfont="no"/>
+<setting alwaysvectorfont="yes"/>
 <setting keepoldvectorfont="yes"/>
 <setting verticaltext="up"/>
@@
 </classes>
 <parts>
-<part name="KT1" library="dp_devices" deviceset="KT0915" device=""/>
+<part name="KT0915" library="dp_devices" deviceset="KT0915" device=""/>
 <part name="GND2" library="SparkFun-Aesthetics" deviceset="GND" device=""/>
 <part name="SUPPLY1" library="supply2" library_urn="urn:adsk.eagle:library:372" deviceset="VCC" device=""/>
@@
 </plain>
 <instances>
-<instance part="KT1" gate="G$1" x="78.74" y="96.52" smashed="yes">
+<instance part="KT0915" gate="G$1" x="78.74" y="96.52" smashed="yes">
 <attribute name="NAME" x="76.2" y="121.92" size="1.27" layer="95"/>
 </instance>
@@
 <net name="N$12" class="0">
 <segment>
-<pinref part="KT1" gate="G$1" pin="RFINP"/>
+<pinref part="KT0915" gate="G$1" pin="RFINP"/>
 <wire x1="59.69" y1="99.06" x2="60.96" y2="99.06" width="0.1524" layer="91"/>
 <wire x1="60.96" y1="99.06" x2="40.64" y2="99.06" width="0.1524" layer="91"/>
@@
 <net name="N$26" class="0">
 <segment>
-<pinref part="KT1" gate="G$1" pin="ROUT"/>
+<pinref part="KT0915" gate="G$1" pin="ROUT"/>
 <wire x1="95.25" y1="88.9" x2="96.52" y2="88.9" width="0.1524" layer="91"/>
 <wire x1="96.52" y1="88.9" x2="142.24" y2="88.9" width="0.1524" layer="91"/>
@@
 <net name="GND" class="0">
 <segment>
-<pinref part="KT1" gate="G$1" pin="AVSS"/>
+<pinref part="KT0915" gate="G$1" pin="AVSS"/>
 <pinref part="GND2" gate="1" pin="GND"/>
 <wire x1="96.52" y1="99.06" x2="127" y2="99.06" width="0.1524" layer="91"/>
@@
 <junction x="162.56" y="83.82"/>
 <junction x="162.56" y="73.66"/>
-<pinref part="KT1" gate="G$1" pin="DVSS"/>
+<pinref part="KT0915" gate="G$1" pin="DVSS"/>
 <wire x1="96.52" y1="83.82" x2="127" y2="83.82" width="0.1524" layer="91"/>
 <wire x1="127" y1="83.82" x2="127" y2="73.66" width="0.1524" layer="91"/>
@@
 <segment>
 <pinref part="GND6" gate="1" pin="GND"/>
-<pinref part="KT1" gate="G$1" pin="RFGND"/>
+<pinref part="KT0915" gate="G$1" pin="RFGND"/>
 <wire x1="40.64" y1="93.98" x2="60.96" y2="93.98" width="0.1524" layer="91"/>
 <junction x="40.64" y="93.98"/>
@@
 <wire x1="15.24" y1="101.6" x2="25.4" y2="101.6" width="0.1524" layer="91"/>
 <wire x1="25.4" y1="101.6" x2="25.4" y2="83.82" width="0.1524" layer="91"/>
-<pinref part="KT1" gate="G$1" pin="SDA"/>
+<pinref part="KT0915" gate="G$1" pin="SDA"/>
 <wire x1="25.4" y1="83.82" x2="33.02" y2="83.82" width="0.1524" layer="91"/>
 <junction x="15.24" y="101.6"/>
@@
 <wire x1="15.24" y1="104.14" x2="27.94" y2="104.14" width="0.1524" layer="91"/>
 <wire x1="27.94" y1="104.14" x2="27.94" y2="88.9" width="0.1524" layer="91"/>
-<pinref part="KT1" gate="G$1" pin="SCL"/>
+<pinref part="KT0915" gate="G$1" pin="SCL"/>
 <wire x1="27.94" y1="88.9" x2="50.8" y2="88.9" width="0.1524" layer="91"/>
 <junction x="15.24" y="104.14"/>
@@
 <pinref part="C2" gate="G$1" pin="1"/>
 <wire x1="119.38" y1="109.22" x2="129.54" y2="109.22" width="0.1524" layer="91"/>
-<pinref part="KT1" gate="G$1" pin="AVDD"/>
+<pinref part="KT0915" gate="G$1" pin="AVDD"/>
 <wire x1="96.52" y1="104.14" x2="114.3" y2="104.14" width="0.1524" layer="91"/>
 <wire x1="114.3" y1="104.14" x2="114.3" y2="109.22" width="0.1524" layer="91"/>
@@
 </segment>
 <segment>
-<pinref part="KT1" gate="G$1" pin="ENABLE"/>
+<pinref part="KT0915" gate="G$1" pin="ENABLE"/>
 <wire x1="60.96" y1="114.3" x2="53.34" y2="114.3" width="0.1524" layer="91"/>
 <wire x1="53.34" y1="114.3" x2="53.34" y2="121.92" width="0.1524" layer="91"/>
@@
 <net name="N$4" class="0">
 <segment>
-<pinref part="KT1" gate="G$1" pin="XI/RCLK"/>
+<pinref part="KT0915" gate="G$1" pin="XI/RCLK"/>
 <wire x1="96.52" y1="109.22" x2="106.68" y2="109.22" width="0.1524" layer="91"/>
 <wire x1="106.68" y1="109.22" x2="106.68" y2="111.76" width="0.1524" layer="91"/>
@@
 <net name="N$5" class="0">
 <segment>
-<pinref part="KT1" gate="G$1" pin="XO"/>
+<pinref part="KT0915" gate="G$1" pin="XO"/>
 <wire x1="96.52" y1="114.3" x2="104.14" y2="114.3" width="0.1524" layer="91"/>
 <wire x1="104.14" y1="114.3" x2="104.14" y2="116.84" width="0.1524" layer="91"/>
@@
 <net name="N$6" class="0">
 <segment>
-<pinref part="KT1" gate="G$1" pin="LOUT"/>
+<pinref part="KT0915" gate="G$1" pin="LOUT"/>
 <wire x1="96.52" y1="93.98" x2="111.76" y2="93.98" width="0.1524" layer="91"/>
 <wire x1="111.76" y1="93.98" x2="111.76" y2="91.44" width="0.1524" layer="91"/>
@@
 <net name="N$9" class="0">
 <segment>
-<pinref part="KT1" gate="G$1" pin="AMINN"/>
+<pinref part="KT0915" gate="G$1" pin="AMINN"/>
 <wire x1="60.96" y1="109.22" x2="48.26" y2="109.22" width="0.1524" layer="91"/>
 <wire x1="48.26" y1="109.22" x2="48.26" y2="124.46" width="0.1524" layer="91"/>
@@
 <net name="N$11" class="0">
 <segment>
-<pinref part="KT1" gate="G$1" pin="AMINP"/>
+<pinref part="KT0915" gate="G$1" pin="AMINP"/>
 <wire x1="60.96" y1="104.14" x2="45.72" y2="104.14" width="0.1524" layer="91"/>
 <wire x1="45.72" y1="104.14" x2="45.72" y2="134.62" width="0.1524" layer="91"/>

Commit message: KT0915 Arduino Library
Changed lines of the file:
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@@
 <wire x1="60.96" y1="99.06" x2="40.64" y2="99.06" width="0.1524" layer="91"/>
 <wire x1="40.64" y1="99.06" x2="40.64" y2="134.62" width="0.1524" layer="91"/>
-<junction x="60.96" y="99.06"/>
 <wire x1="40.64" y1="134.62" x2="30.48" y2="134.62" width="0.1524" layer="91"/>
 <pinref part="ANT2" gate="A" pin="1"/>
@@
 <wire x1="95.25" y1="88.9" x2="96.52" y2="88.9" width="0.1524" layer="91"/>
 <wire x1="96.52" y1="88.9" x2="142.24" y2="88.9" width="0.1524" layer="91"/>
-<junction x="96.52" y="88.9"/>
 <wire x1="142.24" y1="88.9" x2="142.24" y2="81.28" width="0.1524" layer="91"/>
 <pinref part="C5" gate="G$1" pin="1"/>
 <wire x1="142.24" y1="81.28" x2="144.78" y2="81.28" width="0.1524" layer="91"/>
-<junction x="144.78" y="81.28"/>
 </segment>
 </net>
@@
 <wire x1="127" y1="99.06" x2="127" y2="101.6" width="0.1524" layer="91"/>
 <wire x1="127" y1="101.6" x2="129.54" y2="101.6" width="0.1524" layer="91"/>
-<junction x="127" y="99.06"/>
 </segment>
 <segment>
@@
 <pinref part="GND4" gate="1" pin="GND"/>
 <wire x1="162.56" y1="83.82" x2="162.56" y2="73.66" width="0.1524" layer="91"/>
-<junction x="162.56" y="83.82"/>
-<junction x="162.56" y="73.66"/>
 <pinref part="KT0915" gate="G$1" pin="DVSS"/>
 <wire x1="96.52" y1="83.82" x2="127" y2="83.82" width="0.1524" layer="91"/>
 <wire x1="127" y1="83.82" x2="127" y2="73.66" width="0.1524" layer="91"/>
 <wire x1="127" y1="73.66" x2="162.56" y2="73.66" width="0.1524" layer="91"/>
-<junction x="96.52" y="83.82"/>
 </segment>
 <segment>
@@
 <pinref part="KT0915" gate="G$1" pin="RFGND"/>
 <wire x1="40.64" y1="93.98" x2="60.96" y2="93.98" width="0.1524" layer="91"/>
-<junction x="40.64" y="93.98"/>
-<junction x="60.96" y="93.98"/>
-</segment>
-<segment>
-<pinref part="GND1" gate="1" pin="GND"/>
-<pinref part="ARDUINO1" gate="G$1" pin="GND"/>
-<wire x1="-30.48" y1="104.14" x2="-15.24" y2="104.14" width="0.1524" layer="91"/>
-<junction x="-30.48" y="104.14"/>
-<junction x="-15.24" y="104.14"/>
 </segment>
 <segment>
@@
 <wire x1="119.38" y1="144.78" x2="119.38" y2="137.16" width="0.1524" layer="91"/>
 <junction x="119.38" y="137.16"/>
-<junction x="114.3" y="137.16"/>
-<junction x="127" y="137.16"/>
+</segment>
+<segment>
+<pinref part="ARDUINO1" gate="G$1" pin="GND"/>
+<pinref part="GND1" gate="1" pin="GND"/>
+<wire x1="-15.24" y1="104.14" x2="-30.48" y2="104.14" width="0.1524" layer="91"/>
 </segment>
 </net>
@@
 <pinref part="KT0915" gate="G$1" pin="SDA"/>
 <wire x1="25.4" y1="83.82" x2="33.02" y2="83.82" width="0.1524" layer="91"/>
-<junction x="15.24" y="101.6"/>
 <pinref part="R1" gate="G$1" pin="2"/>
 <wire x1="33.02" y1="83.82" x2="60.96" y2="83.82" width="0.1524" layer="91"/>
@@
 <pinref part="KT0915" gate="G$1" pin="SCL"/>
 <wire x1="27.94" y1="88.9" x2="50.8" y2="88.9" width="0.1524" layer="91"/>
-<junction x="15.24" y="104.14"/>
 <pinref part="R2" gate="G$1" pin="2"/>
 <wire x1="50.8" y1="88.9" x2="60.96" y2="88.9" width="0.1524" layer="91"/>
@@
 <pinref part="SUPPLY2" gate="G$1" pin="VCC"/>
 <wire x1="30.48" y1="111.76" x2="30.48" y2="114.3" width="0.1524" layer="91"/>
-<junction x="30.48" y="114.3"/>
 </segment>
 <segment>
@@
 <wire x1="114.3" y1="104.14" x2="114.3" y2="109.22" width="0.1524" layer="91"/>
 <wire x1="114.3" y1="109.22" x2="119.38" y2="109.22" width="0.1524" layer="91"/>
-<junction x="119.38" y="109.22"/>
 <wire x1="129.54" y1="109.22" x2="139.7" y2="109.22" width="0.1524" layer="91"/>
-<junction x="129.54" y="109.22"/>
 <pinref part="SUPPLY1" gate="G$1" pin="VCC"/>
 <wire x1="139.7" y1="109.22" x2="139.7" y2="114.3" width="0.1524" layer="91"/>
@@
 <pinref part="SUPPLY3" gate="G$1" pin="VCC"/>
 <wire x1="68.58" y1="121.92" x2="68.58" y2="124.46" width="0.1524" layer="91"/>
-<junction x="60.96" y="114.3"/>
-<junction x="68.58" y="124.46"/>
 </segment>
 <segment>
@@
 <pinref part="Q1" gate="G$1" pin="2"/>
 <wire x1="121.92" y1="111.76" x2="121.92" y2="116.84" width="0.1524" layer="91"/>
-<junction x="96.52" y="109.22"/>
 <pinref part="C4" gate="G$1" pin="1"/>
 <wire x1="127" y1="129.54" x2="127" y2="116.84" width="0.1524" layer="91"/>
 <wire x1="127" y1="116.84" x2="121.92" y2="116.84" width="0.1524" layer="91"/>
-<junction x="121.92" y="116.84"/>
 </segment>
 </net>
@@
 <pinref part="Q1" gate="G$1" pin="1"/>
 <wire x1="104.14" y1="116.84" x2="106.68" y2="116.84" width="0.1524" layer="91"/>
-<junction x="96.52" y="114.3"/>
 <pinref part="C3" gate="G$1" pin="1"/>
 <wire x1="106.68" y1="116.84" x2="111.76" y2="116.84" width="0.1524" layer="91"/>
@@
 <pinref part="C6" gate="G$1" pin="1"/>
 <wire x1="111.76" y1="91.44" x2="144.78" y2="91.44" width="0.1524" layer="91"/>
-<junction x="96.52" y="93.98"/>
-<junction x="144.78" y="91.44"/>
 </segment>
 </net>
@@
 <pinref part="X1" gate="G$1" pin="2"/>
 <wire x1="152.4" y1="91.44" x2="162.56" y2="91.44" width="0.1524" layer="91"/>
-<junction x="162.56" y="91.44"/>
 </segment>
 </net>
@@
 <pinref part="X1" gate="G$1" pin="3"/>
 <wire x1="157.48" y1="88.9" x2="162.56" y2="88.9" width="0.1524" layer="91"/>
-<junction x="162.56" y="88.9"/>
 </segment>
 </net>
@@
 <pinref part="C7" gate="G$1" pin="2"/>
 <wire x1="55.88" y1="124.46" x2="55.88" y2="127" width="0.1524" layer="91"/>
-<junction x="60.96" y="109.22"/>
-<junction x="55.88" y="127"/>
 </segment>
 </net>
@@
 <pinref part="ANT1" gate="A" pin="1"/>
 <wire x1="48.26" y1="134.62" x2="48.26" y2="142.24" width="0.1524" layer="91"/>
-<junction x="60.96" y="104.14"/>
 <junction x="48.26" y="142.24"/>
 </segment>
