File: extras/schematic/minimal_receiver.sch (EAGLE design)
At the start: 15 parts, among them X1 1501_03

Commit message: KT0915 Arduino Library
Parts:
- added AM, DOWN, FM, UP: (no value), adafruit:SWITCH_PUSHBUTTONEVQ-PE
- C7: value (none) -> 100nF
- renumbered KT1 to KT0915
Connections:
- new net N$1: ARDUINO1.D4, FM.P$2
- new net N$10: AM.P$2, ARDUINO1.D5
- new net N$13: ARDUINO1.D6, UP.P$2
- new net N$14: ARDUINO1.D7, DOWN.P$2
- net GND: now also AM.P$1, DOWN.P$1, FM.P$1, UP.P$1

Commit message: KT0915 Arduino Library
Changed lines of the file:
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@@
 <wire x1="60.96" y1="99.06" x2="40.64" y2="99.06" width="0.1524" layer="91"/>
 <wire x1="40.64" y1="99.06" x2="40.64" y2="134.62" width="0.1524" layer="91"/>
-<junction x="60.96" y="99.06"/>
 <wire x1="40.64" y1="134.62" x2="30.48" y2="134.62" width="0.1524" layer="91"/>
 <pinref part="ANT2" gate="A" pin="1"/>
 <wire x1="30.48" y1="134.62" x2="30.48" y2="142.24" width="0.1524" layer="91"/>
-<junction x="30.48" y="142.24"/>
 </segment>
 </net>
@@
 <wire x1="95.25" y1="88.9" x2="96.52" y2="88.9" width="0.1524" layer="91"/>
 <wire x1="96.52" y1="88.9" x2="142.24" y2="88.9" width="0.1524" layer="91"/>
-<junction x="96.52" y="88.9"/>
 <wire x1="142.24" y1="88.9" x2="142.24" y2="81.28" width="0.1524" layer="91"/>
 <pinref part="C5" gate="G$1" pin="1"/>
 <wire x1="142.24" y1="81.28" x2="144.78" y2="81.28" width="0.1524" layer="91"/>
-<junction x="144.78" y="81.28"/>
 </segment>
 </net>
@@
 <wire x1="127" y1="99.06" x2="127" y2="101.6" width="0.1524" layer="91"/>
 <wire x1="127" y1="101.6" x2="129.54" y2="101.6" width="0.1524" layer="91"/>
-<junction x="127" y="99.06"/>
 </segment>
 <segment>
@@
 <pinref part="GND4" gate="1" pin="GND"/>
 <wire x1="162.56" y1="83.82" x2="162.56" y2="73.66" width="0.1524" layer="91"/>
-<junction x="162.56" y="83.82"/>
-<junction x="162.56" y="73.66"/>
 <pinref part="KT0915" gate="G$1" pin="DVSS"/>
 <wire x1="96.52" y1="83.82" x2="127" y2="83.82" width="0.1524" layer="91"/>
 <wire x1="127" y1="83.82" x2="127" y2="73.66" width="0.1524" layer="91"/>
 <wire x1="127" y1="73.66" x2="162.56" y2="73.66" width="0.1524" layer="91"/>
-<junction x="96.52" y="83.82"/>
 </segment>
 <segment>
@@
 <pinref part="KT0915" gate="G$1" pin="RFGND"/>
 <wire x1="40.64" y1="93.98" x2="60.96" y2="93.98" width="0.1524" layer="91"/>
-<junction x="40.64" y="93.98"/>
-<junction x="60.96" y="93.98"/>
 </segment>
 <segment>
@@
 <pinref part="ARDUINO1" gate="G$1" pin="GND"/>
 <wire x1="-30.48" y1="104.14" x2="-15.24" y2="104.14" width="0.1524" layer="91"/>
-<junction x="-30.48" y="104.14"/>
-<junction x="-15.24" y="104.14"/>
 <pinref part="FM" gate="G$1" pin="P$1"/>
 <pinref part="AM" gate="G$1" pin="P$1"/>
@@
 <pinref part="UP" gate="G$1" pin="P$1"/>
 <wire x1="-35.56" y1="76.2" x2="-35.56" y2="83.82" width="0.1524" layer="91"/>
-<junction x="-35.56" y="83.82"/>
 <pinref part="DOWN" gate="G$1" pin="P$1"/>
 <wire x1="-35.56" y1="68.58" x2="-35.56" y2="76.2" width="0.1524" layer="91"/>
-<junction x="-35.56" y="76.2"/>
 <wire x1="-35.56" y1="91.44" x2="-35.56" y2="104.14" width="0.1524" layer="91"/>
-<junction x="-35.56" y="91.44"/>
 <wire x1="-35.56" y1="104.14" x2="-30.48" y2="104.14" width="0.1524" layer="91"/>
 </segment>
@@
 <wire x1="119.38" y1="144.78" x2="119.38" y2="137.16" width="0.1524" layer="91"/>
 <junction x="119.38" y="137.16"/>
-<junction x="114.3" y="137.16"/>
-<junction x="127" y="137.16"/>
 </segment>
 </net>
@@
 <pinref part="KT0915" gate="G$1" pin="SDA"/>
 <wire x1="25.4" y1="83.82" x2="33.02" y2="83.82" width="0.1524" layer="91"/>
-<junction x="15.24" y="101.6"/>
 <pinref part="R1" gate="G$1" pin="2"/>
 <wire x1="33.02" y1="83.82" x2="60.96" y2="83.82" width="0.1524" layer="91"/>
@@
 <pinref part="KT0915" gate="G$1" pin="SCL"/>
 <wire x1="27.94" y1="88.9" x2="50.8" y2="88.9" width="0.1524" layer="91"/>
-<junction x="15.24" y="104.14"/>
 <pinref part="R2" gate="G$1" pin="2"/>
 <wire x1="50.8" y1="88.9" x2="60.96" y2="88.9" width="0.1524" layer="91"/>
@@
 <pinref part="SUPPLY2" gate="G$1" pin="VCC"/>
 <wire x1="30.48" y1="111.76" x2="30.48" y2="114.3" width="0.1524" layer="91"/>
-<junction x="30.48" y="114.3"/>
 </segment>
 <segment>
@@
 <wire x1="114.3" y1="104.14" x2="114.3" y2="109.22" width="0.1524" layer="91"/>
 <wire x1="114.3" y1="109.22" x2="119.38" y2="109.22" width="0.1524" layer="91"/>
-<junction x="119.38" y="109.22"/>
 <wire x1="129.54" y1="109.22" x2="139.7" y2="109.22" width="0.1524" layer="91"/>
-<junction x="129.54" y="109.22"/>
 <pinref part="SUPPLY1" gate="G$1" pin="VCC"/>
 <wire x1="139.7" y1="109.22" x2="139.7" y2="114.3" width="0.1524" layer="91"/>
-<junction x="139.7" y="114.3"/>
 </segment>
 <segment>
@@
 <pinref part="SUPPLY3" gate="G$1" pin="VCC"/>
 <wire x1="68.58" y1="121.92" x2="68.58" y2="124.46" width="0.1524" layer="91"/>
-<junction x="60.96" y="114.3"/>
-<junction x="68.58" y="124.46"/>
 </segment>
 <segment>
@@
 <pinref part="Q1" gate="G$1" pin="2"/>
 <wire x1="121.92" y1="111.76" x2="121.92" y2="116.84" width="0.1524" layer="91"/>
-<junction x="96.52" y="109.22"/>
 <pinref part="C4" gate="G$1" pin="1"/>
 <wire x1="127" y1="129.54" x2="127" y2="116.84" width="0.1524" layer="91"/>
 <wire x1="127" y1="116.84" x2="121.92" y2="116.84" width="0.1524" layer="91"/>
-<junction x="121.92" y="116.84"/>
 </segment>
 </net>
@@
 <pinref part="Q1" gate="G$1" pin="1"/>
 <wire x1="104.14" y1="116.84" x2="106.68" y2="116.84" width="0.1524" layer="91"/>
-<junction x="96.52" y="114.3"/>
 <pinref part="C3" gate="G$1" pin="1"/>
 <wire x1="106.68" y1="116.84" x2="111.76" y2="116.84" width="0.1524" layer="91"/>
@@
 <pinref part="C6" gate="G$1" pin="1"/>
 <wire x1="111.76" y1="91.44" x2="144.78" y2="91.44" width="0.1524" layer="91"/>
-<junction x="96.52" y="93.98"/>
-<junction x="144.78" y="91.44"/>
 </segment>
 </net>
@@
 <pinref part="X1" gate="G$1" pin="2"/>
 <wire x1="152.4" y1="91.44" x2="162.56" y2="91.44" width="0.1524" layer="91"/>
-<junction x="162.56" y="91.44"/>
 </segment>
 </net>
@@
 <pinref part="X1" gate="G$1" pin="3"/>
 <wire x1="157.48" y1="88.9" x2="162.56" y2="88.9" width="0.1524" layer="91"/>
-<junction x="162.56" y="88.9"/>
 </segment>
 </net>
@@
 <pinref part="C7" gate="G$1" pin="2"/>
 <wire x1="55.88" y1="124.46" x2="55.88" y2="127" width="0.1524" layer="91"/>
-<junction x="60.96" y="109.22"/>
-<junction x="55.88" y="127"/>
 </segment>
 </net>
@@
 <pinref part="ANT1" gate="A" pin="1"/>
 <wire x1="48.26" y1="134.62" x2="48.26" y2="142.24" width="0.1524" layer="91"/>
-<junction x="60.96" y="104.14"/>
-<junction x="48.26" y="142.24"/>
-</segment>
-</net>
+</segment>
+</net>
